File: hardware/schematic/Full_Schematic.sch (EAGLE design)
At the start: 222 parts, among them Q1 SS8050-G, Q2 SS8050-G, SW3 1825910-6, SW4 1825910-6, SW5 1825910-6, U14 MMSZ5225BT1G, U15 MMSZ5230BT1G, U16 MMSZ5225BT1G, U19 LM358DR

Commit message: Schematic updates
Connections:
- removed net 0: 19_PINOUT.19, 4PIN_I2C_TEST.4, C3.3OUT1.2, C3.3OUT10.2, C3.3OUT11.1, C3.3OUT12.1, C3.3OUT2.2, C3.3OUT3.1, C3.3OUT4.1, C3.3OUT5.2, C3.3OUT6.2, C3.3OUT7.1, C3.3OUT8.1, C3.3OUT9.2, CBUS.2, CENS.2, CENS1.2, CUSB.2, CUSB1.1, CUSB2.1, CUSB3.2, CUSB4.2, CUSB5.2, CUSB6.2, CVCCSERVO.2, CVINT.2, CVMOT.1, CVMOT2.1, CVMOT3.1, CVMOT4.1, D10.K, D11.K, D12.K, D14.K, D15.K, D16.K, D18.K, D19.K, D2.K, D20.K, D3.K, D4.K, D6.K, D7.K, D8.K, I2C_USBC_IN.GND, I2C_USBC_IN.GND_2, I2C_USBC_OUT.GND, I2C_USBC_OUT.GND_2, PURESET.1, R1.A, RADECAY.2, RAISEN.2, RBDECAY.2, RBISEN.2, RILIM.1, RILIM1.1, RILIM2.1, ROE.2, RS.1, RS1.1, RS2.1, RS3.1, RS4.1, RS5.1, RS6.1, RU1.1, RU3.1, RUSB.2, RUSB1.2, RUSB2.2, RUSB3.2, RUSB4.2, RUSB5.2, RUSB6.2, RUSB7.2, RUSB8.2, RUSB9.2, SENCDC1.2, SENCDC2.2, SENSOR1.GND, SENSOR2.GND, SENSOR3.GND, SENSOR4.GND, SENSOR5.GND, SENSOR_MUX.!RESET, SENSOR_MUX.A1, SENSOR_MUX.A2, SENSOR_MUX.GND, SENSOR_PSWITCH.GND, SENSOR_USBA_IN.4, SENSOR_USBA_OUT.4, SERVO_CONTROLLER.EXTCLK, SERVO_CONTROLLER.VSS, SERVO_PINOUT.11, SERVO_PINOUT.5, SERVO_PINOUT.6, SERVO_PSWITCH.GND, SERVO_REGULATOR.GND, STEPPER_CONTROLLER.EXP(GND), STEPPER_CONTROLLER.GND, STEPPER_P_SWITCH.GND, STEPPER_REGULATOR.GND, STEPPER_USBC_IN.GND, STEPPER_USBC_IN.GND_2, STEPPER_USBC_OUT.GND, STEPPER_USBC_OUT.GND_2, SW3.3, SW3.4, SW4.1, SW5.1, U$3.GND, U$4.GND, U$5.GND, U16.ANODE, U19.GND, UART_USBC_IN.GND, UART_USBC_IN.GND_2, UART_USB_CONVERTER.GND
- net GND: now also 19_PINOUT.19, 4PIN_I2C_TEST.4, C3.3OUT1.2, C3.3OUT10.2, C3.3OUT11.1, C3.3OUT12.1, C3.3OUT2.2, C3.3OUT3.1, C3.3OUT4.1, C3.3OUT5.2, C3.3OUT6.2, C3.3OUT7.1, C3.3OUT8.1, C3.3OUT9.2, CBUS.2, CENS.2, CENS1.2, CUSB.2, CUSB1.1, CUSB2.1, CUSB3.2, CUSB4.2, CUSB5.2, CUSB6.2, CVCCSERVO.2, CVINT.2, CVMOT.1, CVMOT2.1, CVMOT3.1, CVMOT4.1, D10.K, D11.K, D12.K, D14.K, D15.K, D16.K, D18.K, D19.K, D2.K, D20.K, D3.K, D4.K, D6.K, D7.K, D8.K, I2C_USBC_IN.GND, I2C_USBC_IN.GND_2, I2C_USBC_OUT.GND, I2C_USBC_OUT.GND_2, PURESET.1, R1.A, RADECAY.2, RAISEN.2, RBDECAY.2, RBISEN.2, RILIM.1, RILIM1.1, RILIM2.1, ROE.2, RS.1, RS1.1, RS2.1, RS3.1, RS4.1, RS5.1, RS6.1, RU1.1, RU3.1, RUSB.2, RUSB1.2, RUSB2.2, RUSB3.2, RUSB4.2, RUSB5.2, RUSB6.2, RUSB7.2, RUSB8.2, RUSB9.2, SENCDC1.2, SENCDC2.2, SENSOR1.GND, SENSOR2.GND, SENSOR3.GND, SENSOR4.GND, SENSOR5.GND, SENSOR_MUX.!RESET, SENSOR_MUX.A1, SENSOR_MUX.A2, SENSOR_MUX.GND, SENSOR_PSWITCH.GND, SENSOR_USBA_IN.4, SENSOR_USBA_OUT.4, SERVO_CONTROLLER.EXTCLK, SERVO_CONTROLLER.VSS, SERVO_PINOUT.11, SERVO_PINOUT.5, SERVO_PINOUT.6, SERVO_PSWITCH.GND, SERVO_REGULATOR.GND, STEPPER_CONTROLLER.EXP(GND), STEPPER_CONTROLLER.GND, STEPPER_P_SWITCH.GND, STEPPER_REGULATOR.GND, STEPPER_USBC_IN.GND, STEPPER_USBC_IN.GND_2, STEPPER_USBC_OUT.GND, STEPPER_USBC_OUT.GND_2, SW3.3, SW3.4, SW4.1, SW5.1, U$3.GND, U$4.GND, U$5.GND, U16.ANODE, U19.GND, UART_USBC_IN.GND, UART_USBC_IN.GND_2, UART_USB_CONVERTER.GND

Commit message: Schematic Updates
Connections:
- net N$60 renamed 3.3USBA
Other:
- note added: "Connector and Pinout"
- note added: "MCU"
- note added: "Power Swtiches"
- note added: "Regulators"
- note added: "SD Connector"
- note added: "Sensors and Mux"
- note added: "Servo Motors Control"
- note added: "Stepper Motor Control"
- note added: "UART-USB Converter"
- moved on the sheet: 19_PINOUT, 3.3V_REGULATOR, 4PIN_I2C_TEST, 5V_REGULATOR, BAT_JP, C3.3MCU, C3.3MCU1, C3.3OUT1, C3.3OUT10, C3.3OUT11, C3.3OUT12, C3.3OUT2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
