File: hardware/schematic/PCB_Sensors.sch (EAGLE design)
At the start: 22 parts, among them U1 VEML7700-TT, U2 VEML7700-TT, U3 VEML7700-TT, U4 VEML7700-TT, U5 VEML7700-TT, U6 TCA9548APWR

Commit message: Schematic Updates
Parts:
- removed U1, U2, U3, U4, U5: VEML7700-TT, VEML7700-TT:VEML7700-TT
- removed U6: TCA9548APWR, TCA9548APWR:TCA9548APWR
- removed USBASEN: USB-AP-S-RA-SMT, USB-AP-S-RA-SMT:USB-AP-S-RA-SMT
- added SENSOR1, SENSOR2, SENSOR3, SENSOR4, SENSOR5: VEML7700-TT, VEML7700-TT:VEML7700-TT
- added SENSOR_MUX: TCA9548APWR, TCA9548APWR:TCA9548APWR
- added SENSOR_USBA_OUT: USB-AP-S-RA-SMT, USB-AP-S-RA-SMT:USB-AP-S-RA-SMT
- added SW3: 1825910-6, 1825910-6:1825910-6
Connections:
- removed net 0: SENCDC1.2, SENCDC2.2, U1.GND, U2.GND, U3.GND, U4.GND, U5.GND, U6.A0, U6.A1, U6.A2, U6.GND
- removed net MCUI2CRESET: PURESET.1, PUSCL.1, U6.!RESET, USBASEN.4
- new net GND: PURESET.1, SENCDC1.2, SENCDC2.2, SENSOR1.GND, SENSOR2.GND, SENSOR3.GND, SENSOR4.GND, SENSOR5.GND, SENSOR_MUX.!RESET, SENSOR_MUX.A1, SENSOR_MUX.A2, SENSOR_MUX.GND, SENSOR_USBA_OUT.4, SW3.3, SW3.4
- net 3.3OUTCON: now also SENSOR1.VDD, SENSOR2.VDD, SENSOR3.VDD, SENSOR4.VDD, SENSOR5.VDD, SENSOR_MUX.A0, SENSOR_MUX.VCC, SENSOR_USBA_OUT.1, SW3.1, SW3.2; no longer U1.VDD, U2.VDD, U3.VDD, U4.VDD, U5.VDD, U6.VCC, USBASEN.1
- net MCUI2CSCL: now also PUSCL.1, SENSOR_MUX.SCL, SENSOR_USBA_OUT.3; no longer U6.SCL, USBASEN.3
- net MCUI2CSDA: now also SENSOR_MUX.SDA, SENSOR_USBA_OUT.2; no longer U6.SDA, USBASEN.2
- net MUXSC0: now also SENSOR1.SCL, SENSOR_MUX.SC0; no longer U1.SCL, U6.SC0
- net MUXSC1: now also SENSOR2.SCL, SENSOR_MUX.SC1; no longer U2.SCL, U6.SC1
- net MUXSC2: now also SENSOR3.SCL, SENSOR_MUX.SC2; no longer U3.SCL, U6.SC2
- net MUXSC3: now also SENSOR4.SCL, SENSOR_MUX.SC3; no longer U4.SCL, U6.SC3
- net MUXSC4: now also SENSOR5.SCL, SENSOR_MUX.SC4; no longer U5.SCL, U6.SC4
- net MUXSD0: now also SENSOR1.SDA, SENSOR_MUX.SD0; no longer U1.SDA, U6.SD0
- net MUXSD1: now also SENSOR2.SDA, SENSOR_MUX.SD1; no longer U2.SDA, U6.SD1
- net MUXSD2: now also SENSOR3.SDA, SENSOR_MUX.SD2; no longer U3.SDA, U6.SD2
- net MUXSD3: now also SENSOR4.SDA, SENSOR_MUX.SD3; no longer U4.SDA, U6.SD3
- net MUXSD4: now also SENSOR5.SDA, SENSOR_MUX.SD4; no longer U5.SDA, U6.SD4
Other:
- note added: "Sensors and Mux"
- moved on the sheet: PURESET, PUSC0, PUSC1, PUSC2, PUSC3, PUSC4, PUSCL, PUSD0, PUSD1, PUSD2, PUSD3, PUSD4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

Commit message: Schematics updates
Changed lines of the file:
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@@
 <part name="SENSOR5" library="VEML7700-TT" deviceset="VEML7700-TT" device=""/>
 <part name="SENSOR_MUX" library="TCA9548APWR" deviceset="TCA9548APWR" device=""/>
-<part name="X_1" library="ngspice-simulation" library_urn="urn:adsk.eagle:library:527439" deviceset="GND" device=""/>
 <part name="PUSC0" library="rcl" library_urn="urn:adsk.eagle:library:334" deviceset="R-US_" device="M0805" package3d_urn="urn:adsk.eagle:package:23556/2" value="2.2k"/>
 <part name="PUSC1" library="rcl" library_urn="urn:adsk.eagle:library:334" deviceset="R-US_" device="M0805" package3d_urn="urn:adsk.eagle:package:23556/2" value="2.2k"/>
@@
 <part name="PUSD3" library="rcl" library_urn="urn:adsk.eagle:library:334" deviceset="R-US_" device="M0805" package3d_urn="urn:adsk.eagle:package:23556/2" value="2.2k"/>
 <part name="PUSD4" library="rcl" library_urn="urn:adsk.eagle:library:334" deviceset="R-US_" device="M0805" package3d_urn="urn:adsk.eagle:package:23556/2" value="2.2k"/>
-<part name="X_2" library="ngspice-simulation" library_urn="urn:adsk.eagle:library:527439" deviceset="GND" device=""/>
 <part name="PURESET" library="rcl" library_urn="urn:adsk.eagle:library:334" deviceset="R-US_" device="M0805" package3d_urn="urn:adsk.eagle:package:23556/2" value="2.2k"/>
 <part name="PUSCL" library="rcl" library_urn="urn:adsk.eagle:library:334" deviceset="R-US_" device="M0805" package3d_urn="urn:adsk.eagle:package:23556/2" value="2.2k"/>
@@
 <part name="SENCDC2" library="rcl" library_urn="urn:adsk.eagle:library:334" deviceset="C-EU" device="C0805" package3d_urn="urn:adsk.eagle:package:23617/2" value="200pF"/>
 <part name="SW3" library="1825910-6" deviceset="1825910-6" device=""/>
+<part name="SUPPLY1" library="supply2" library_urn="urn:adsk.eagle:library:372" deviceset="GND" device=""/>
+<part name="SUPPLY2" library="supply2" library_urn="urn:adsk.eagle:library:372" deviceset="GND" device=""/>
 </parts>
 <sheets>
@@
 <attribute name="VALUE" x="-58.42" y="-24.32" size="2.0828" layer="96" ratio="10" rot="SR0"/>
 </instance>
-<instance part="X_1" gate="G$1" x="132.08" y="-58.42" smashed="yes"/>
 <instance part="PUSC0" gate="G$1" x="81.28" y="61.976" smashed="yes" rot="R90">
 <attribute name="NAME" x="79.7814" y="58.166" size="1.778" layer="95" rot="R90"/>
@@
 <attribute name="VALUE" x="92.202" y="-38.354" size="1.778" layer="96" rot="R90"/>
 </instance>
-<instance part="X_2" gate="G$1" x="-20.32" y="-43.18" smashed="yes"/>
 <instance part="PURESET" gate="G$1" x="-121.92" y="61.976" smashed="yes" rot="R90">
 <attribute name="NAME" x="-123.4186" y="58.166" size="1.778" layer="95" rot="R90"/>
@@
 <attribute name="NAME" x="-96.5297" y="-17.00685" size="1.803440625" layer="95"/>
 <attribute name="VALUE" x="-96.528309375" y="-30.49246875" size="1.802940625" layer="96"/>
+</instance>
+<instance part="SUPPLY1" gate="GND" x="-20.32" y="-45.72" smashed="yes">
+<attribute name="VALUE" x="-22.225" y="-48.895" size="1.778" layer="96"/>
+</instance>
+<instance part="SUPPLY2" gate="GND" x="132.08" y="-60.96" smashed="yes">
+<attribute name="VALUE" x="130.175" y="-64.135" size="1.778" layer="96"/>
 </instance>
 </instances>
@@
 <wire x1="116.84" y1="-50.8" x2="132.08" y2="-50.8" width="0.1524" layer="91"/>
 <junction x="132.08" y="-50.8"/>
-<pinref part="X_1" gate="G$1" pin="0"/>
+<pinref part="SUPPLY2" gate="GND" pin="GND"/>
 </segment>
 <segment>
@@
 <wire x1="-27.94" y1="-17.78" x2="-20.32" y2="-17.78" width="0.1524" layer="91"/>
 <wire x1="-20.32" y1="-17.78" x2="-20.32" y2="-38.1" width="0.1524" layer="91"/>
-<pinref part="X_2" gate="G$1" pin="0"/>
 <pinref part="SENCDC1" gate="G$1" pin="2"/>
 <wire x1="-20.32" y1="-38.1" x2="-20.32" y2="-43.18" width="0.1524" layer="91"/>
@@
 <wire x1="-66.04" y1="20.32" x2="-66.04" y2="-38.1" width="0.1524" layer="91"/>
 <junction x="-66.04" y="-38.1"/>
+<pinref part="SUPPLY1" gate="GND" pin="GND"/>
 </segment>
 </net>
@@
 </sheet>
 </sheets>
+<errors>
+</errors>
 </schematic>
 </drawing>
