File: hardware/schematic/Servo.brd (EAGLE design)
At the start: 49.5 x 35.2 mm, 23 parts

Commit message: Servo Updated
Parts:
- moved RS 23.2 mm to (44.5, 7.62), turned to 90 degrees
- moved ROE 18.9 mm to (40.6, 7.62), turned to 270 degrees
- moved D9 11.2 mm to (21.1, 21.5), turned to 180 degrees
- moved RUSB4 10.9 mm to (16.5, 25.4)
- moved LED4 10.2 mm to (22.9, 15.2), turned to 180 degrees
- moved RUSB5 6.35 mm to (11.4, 25.4)
- moved RS2 2.84 mm to (24.1, 10.2)
- moved D12 2.54 mm to (14.0, 21.6)
- moved RS3 2.54 mm to (16.5, 6.35)
- moved CUSB4 2.54 mm to (29.2, 25.4)
- moved RS1 2.54 mm to (24.1, 7.62)
- moved RS4 1.27 mm to (16.5, 8.89)
- moved D10 1.27 mm to (11.4, 21.6)
Routing:
- net GND: track 184.8 -> 0.00 mm
- net SRVSDAM: track 62.0 -> 20.2 mm
- net 3.3VOUTUSB1: track 26.6 -> 55.4 mm
- net SRVSCLM: track 50.8 -> 22.3 mm, vias 4 -> 0
- net VBUS12: track 16.6 -> 32.1 mm, vias 2 -> 0
- net A5: track 21.7 -> 9.31 mm
- net CC1_RUSB4: track 19.1 -> 9.43 mm, vias 2 -> 0
- net OE: track 14.3 -> 5.23 mm
- net CC2: track 10.2 -> 3.51 mm, vias 2 -> 0
- net LED_RS6: track 0.00 -> 5.56 mm
- net 5VOUTUSB12: track 64.1 -> 59.4 mm, vias 1 -> 0
- net A2: track 20.2 -> 16.2 mm
- net A3: track 7.67 -> 5.12 mm
- net A4: track 8.76 -> 6.22 mm
- net A1: track 16.6 -> 14.7 mm
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- added copper zone on layer 1, net GND
