File: hardware/schematic/PCB_MCU.brd (EAGLE design)
At the start: 142.2 x 169.8 mm, 131 parts, among them Q1 SS8050-G, Q2 SS8050-G, SW4 1825910-6, SW5 1825910-6, U14 MMSZ5225BT1G, U15 MMSZ5230BT1G

Commit message: Added regulators and SD Card. Needs major work
Parts:
- moved RLEDOUT9 211.8 mm to (43.2, 92.7), turned to 270 degrees
- moved COUT5 208.9 mm to (35.6, 97.8), turned to 90 degrees
- moved COUT4 204.1 mm to (38.1, 97.8), turned to 90 degrees
- moved RLEDOUT 203.7 mm to (38.1, 92.7), turned to 90 degrees
- moved RSDCS 203.2 mm to (27.9, 31.8), turned to 90 degrees
- moved RLEDOUT8 202.6 mm to (40.6, 80.0), turned to 90 degrees
- moved COUT2 199.5 mm to (36.8, 72.4), turned to 270 degrees
- moved COUT3 199.3 mm to (40.6, 97.8), turned to 90 degrees
- moved CINX1 198.4 mm to (12.7, 69.8), turned to 270 degrees
- moved COUT1 195.0 mm to (39.4, 72.4), turned to 270 degrees
- moved DA_CONVERTER_SD 189.8 mm to (21.6, 39.4)
- moved CIN4 189.8 mm to (5.08, 88.9), turned to 270 degrees
- moved RLEDOUT3 189.6 mm to (38.1, 80.0), turned to 270 degrees
- moved CIN2 187.2 mm to (2.54, 69.8), turned to 270 degrees
- moved OP_AMP_LEDS 186.8 mm to (39.4, 86.4), turned to 270 degrees
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Connections:
- net N$1 renamed BOOT_3VREG
- net N$10 renamed TXD_UART_CONV
- net N$11 renamed BOOT_5VREG
- net N$12 renamed RXD_UART_CONV
- net N$13 renamed SW_5VREG
- net N$14 renamed VCC_5VREG
- net N$15 renamed PGOOD_5VREG
- net N$16 renamed MODE_5VREG
- net N$17 renamed TRIP_5VREG
- net N$18 renamed SS_REFIN_5VREG
- net N$19 renamed EN_5VREG
- net N$2 renamed SW_3VREG
- net N$20 renamed LED3_RLED9
- net N$22 renamed FB_5VREG
- net N$26 renamed SUSPEND
- net N$3 renamed VCC_3VREG
- net N$4 renamed PGOOD_3VREG
- net N$40 renamed RST_UART_CONV
- net N$41 renamed VBUS_UART_CONV
- net N$5 renamed EN_3VREG
- net N$52 renamed 3V3_MCU
- net N$53 renamed CC1_UART
- net N$54 renamed LED1_RSDCS
- net N$55 renamed LED_CONVERTER
- net N$56 renamed CC2_UART
- net N$57 renamed SD_CLK
- net N$58 renamed ILIM_SENSOR_S
- net N$59 renamed DATA_I_SD
- net N$6 renamed MODE_3VREG
- net N$60 renamed 3.3USBA
- net N$61 renamed FAULT_SENSOR_S
- net N$62 renamed CC1_I2C
- net N$63 renamed CC2_I2C
- net N$66 renamed CC1_STEPPER
- net N$67 renamed ILIM_SERVO_S
- net N$68 renamed FAULT_SERVO_S
- net N$69 renamed CC2_STEPPER
- net N$7 renamed TRIP_3VREG
- net N$70 renamed ILIM_STEPPER_S
- net N$71 renamed FAULT_STEPPER_S
- net N$74 renamed 2+I_OP_AMP
- net N$75 renamed 2-I_OP_AMP
- net N$76 renamed 2O_OP_AMP
- net N$77 renamed 1I+_OP_AMP
- net N$78 renamed 1I-_OP_AMP
- net N$79 renamed 1O_OP_AMP
- net N$8 renamed SS_REFIN_3VREG
- net N$80 renamed LED2_RLED8
- net N$81 renamed DSR_NC
- net N$86 renamed CTS_NC
- net N$9 renamed FB_3VREG
- net N$91 renamed 5ASD
- net N$92 renamed 6ASD
- removed net 0: 19_PINOUT.19, 4PIN_I2C_TEST.4, C3.3OUT1.2, C3.3OUT10.2, C3.3OUT11.1, C3.3OUT12.1, C3.3OUT2.2, C3.3OUT3.1, C3.3OUT4.1, C3.3OUT5.2, C3.3OUT6.2, C3.3OUT7.1, C3.3OUT8.1, C3.3OUT9.2, CBUS.2, CENS.2, CENS1.2, CUSB.2, CUSB1.1, CUSB2.1, CUSB3.2, CUSB5.2, D14.1, D15.1, D16.1, D2.1, D3.1, D4.1, D6.1, D7.1, D8.1, I2C_USBC_IN.A1-B12, I2C_USBC_IN.A12-B1, RILIM.1, RILIM1.1, RILIM2.1, RU1.1, RU3.1, RUSB.2, RUSB1.2, RUSB2.2, RUSB3.2, RUSB6.2, RUSB7.2, SENSOR_PSWITCH.2, SENSOR_USBA_IN.4, SERVO_PSWITCH.2, STEPPER_P_SWITCH.2, STEPPER_USBC_IN.A1-B12, STEPPER_USBC_IN.A12-B1, SW4.1, SW5.1, UART_USBC_IN.A1-B12, UART_USBC_IN.A12-B1, UART_USB_CONVERTER.29, UART_USB_CONVERTER.3
- net GND: now also 19_PINOUT.19, 4PIN_I2C_TEST.4, C3.3OUT1.2, C3.3OUT10.2, C3.3OUT11.1, C3.3OUT12.1, C3.3OUT2.2, C3.3OUT3.1, C3.3OUT4.1, C3.3OUT5.2, C3.3OUT6.2, C3.3OUT7.1, C3.3OUT8.1, C3.3OUT9.2, CBUS.2, CENS.2, CENS1.2, CUSB.2, CUSB1.1, CUSB2.1, CUSB3.2, CUSB5.2, D14.1, D15.1, D16.1, D2.1, D3.1, D4.1, D6.1, D7.1, D8.1, I2C_USBC_IN.A1-B12, I2C_USBC_IN.A12-B1, RILIM.1, RILIM1.1, RILIM2.1, RU1.1, RU3.1, RUSB.2, RUSB1.2, RUSB2.2, RUSB3.2, RUSB6.2, RUSB7.2, SENSOR_PSWITCH.2, SENSOR_USBA_IN.4, SERVO_PSWITCH.2, STEPPER_P_SWITCH.2, STEPPER_USBC_IN.A1-B12, STEPPER_USBC_IN.A12-B1, SW4.1, SW5.1, UART_USBC_IN.A1-B12, UART_USBC_IN.A12-B1, UART_USB_CONVERTER.29, UART_USB_CONVERTER.3
Other:
- board size 142.2 x 169.8 mm -> 84.8 x 106.7 mm
