File: hardware/schematic/Eagle/Servo.brd (EAGLE design)
At the start: 49.5 x 35.2 mm, 23 parts

Commit message: Updates Schematic
Parts:
- moved D11 30.9 mm to (39.4, 16.5), turned to 180 degrees
- moved D12 25.4 mm to (39.4, 21.6), turned to 180 degrees
- moved CUSB4 21.6 mm to (10.2, 15.2)
- moved SERVO_REGULATOR 15.3 mm to (27.9, 26.7), turned to 90 degrees
- moved RS6 10.2 mm to (26.7, 15.2)
- moved D10 9.25 mm to (8.89, 30.5), turned to 270 degrees
- moved D9 9.16 mm to (16.0, 29.1)
- moved ROE 8.89 mm to (31.8, 7.62)
- moved RS 8.89 mm to (35.6, 7.62)
- moved LED4 8.03 mm to (30.5, 17.8), turned to 90 degrees
- moved RS1 7.73 mm to (16.5, 6.35)
- moved RS2 7.73 mm to (16.5, 8.89)
- moved RUSB4 6.84 mm to (10.2, 27.9)
- moved RS3 6.35 mm to (10.2, 6.35)
- moved RS4 6.35 mm to (10.2, 8.89)
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Routing:
- net SRVSDAM: track 20.2 -> 91.9 mm
- net SRVSCLM: track 22.3 -> 62.1 mm
- net 3.3VOUTUSB1: track 55.4 -> 36.4 mm
- net VBUS12: track 32.1 -> 14.3 mm
- net 5VOUTUSB12: track 59.4 -> 47.1 mm
- net CC1_RUSB4: track 9.43 -> 2.05 mm
- net PWM3: track 29.0 -> 22.7 mm
- net PWM2: track 30.5 -> 24.2 mm
- net PWM1: track 26.3 -> 19.9 mm
- net OE: track 5.23 -> 2.69 mm
- net A5: track 9.31 -> 6.77 mm
- net A3: track 5.12 -> 7.24 mm
- net A4: track 6.22 -> 8.01 mm
- net CC2: track 3.51 -> 2.36 mm
- net A0: track 14.1 -> 13.3 mm
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Other:
- board size 49.5 x 35.2 mm -> 41.9 x 34 mm
